File: rcbus-parallel.kicad_pcb (KiCad board)
At the start: 2 copper layers, 100 x 50 mm, 14 parts, among them J2 Conn_02x20_Odd_Even, P1 Conn_01x39, SW1 SW_DIP_x06, U1 82C55A_PLCC, U2 74HCT688, U3 74HCT04

Commit message: add git submodule library and kibot build stuff
Parts:
- added G3: Symbol_CreativeCommons_Silk_Type2_Small, electrified:Symbol_CreativeCommons_Silk_Type2_Small, B.Cu at (105.3, 157.8)
- added G4: Symbol_CC-Attribution_Silk_Small, electrified:Symbol_CC-Attribution_Silk_Small, B.Cu at (99.3, 157.8)
- added G5: Symbol_CC-ShareAlike_Silk_Small, electrified:Symbol_CC-ShareAlike_Silk_Small, B.Cu at (93.3, 157.8)
- added H1: MountingHole, MountingHole:MountingHole_3.2mm_M3, F.Cu at (68.4, 132.3)
- added R1: 270R, Resistor_THT:R_Axial_DIN0207_L6.3mm_D2.5mm_P7.62mm_Horizontal, F.Cu at (115.5, 120.5)
- moved R4 3.81 mm to (115.6, 131.4)
- moved R2 3.81 mm to (115.6, 123.8)
- moved R3 3.81 mm to (115.6, 127.6)
Other:
- board text added: "2017-2026 Ed Brindley"
- board text added: "CC BY-SA https://creativecommons.org"
- board text added: "Rev: ${VERSION} ${GIT_HASH}"
- board text removed: "2017-2022 Ed Brindley"
- board text removed: "Rev 3-pre"

Commit message: reorg and routing
Parts:
- removed D1: LED, LED_THT:LED_D3.0mm
- removed R1: 270R, Resistor_THT:R_Axial_DIN0207_L6.3mm_D2.5mm_P7.62mm_Horizontal
- removed SW1: SW_DIP_x06, Button_Switch_THT:SW_DIP_SPSTx06_Slide_9.78x17.42mm_W7.62mm_P2.54mm
- added J1: Conn_02x06_Odd_Even, Connector_PinHeader_2.54mm:PinHeader_2x06_P2.54mm_Vertical, F.Cu at (62.6, 140.0)
- J2: footprint Connector_PinHeader_2.54mm:PinHeader_2x13_P2.54mm_Horizontal -> Connector_IDC:IDC-Header_2x13_P2.54mm_Horizontal
- U1: footprint Package_LCC:PLCC-44 -> Package_LCC:PLCC-44_THT-Socket
- moved C1 29.0 mm to (77.9, 123.5)
- moved U3 29.0 mm to (78.5, 134.9)
- moved RN1 16.5 mm to (70.4, 156.4), turned to 90 degrees
- moved R3 16.5 mm to (100.6, 134.4)
- moved R2 15.4 mm to (100.6, 127.3)
- moved R4 15.0 mm to (100.6, 130.8)
- moved C3 11.4 mm to (118.5, 153.9), turned to 180 degrees
- moved J2 7.69 mm to (145.8, 122.7)
- moved U1 5.95 mm to (132.1, 139.3)
- moved U2 4.98 mm to (78.5, 152.0)
- moved C2 4.95 mm to (77.9, 141.0)
Routing:
- net VCC: track 0.00 -> 114.2 mm
- net GND: track 0.00 -> 98.1 mm
- net /RESET: track 0.00 -> 59.4 mm
- net /~{PIO_CS}: track 0.00 -> 59.3 mm
- net /~{IORQ}: track 0.00 -> 54.1 mm, vias 0 -> 1
- net /A1: track 0.00 -> 51.9 mm
- net /~{RESET}: track 0.00 -> 45.9 mm
- net Net-(J1-Pin_4): track 0.00 -> 45.1 mm
- net /A0: track 0.00 -> 44.2 mm
- net Net-(J1-Pin_8): track 0.00 -> 42.6 mm
- net Net-(J1-Pin_6): track 0.00 -> 42.3 mm
- net Net-(J1-Pin_10): track 0.00 -> 40.7 mm
- net /PC3: track 0.00 -> 39.2 mm
- net Net-(J1-Pin_12): track 0.00 -> 38.8 mm
- net /~{RD}: track 0.00 -> 37.3 mm, vias 0 -> 1
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- added copper zone on F.Cu, net GND
Other:
- board text added: "${GIT_HASH}"
- board text added: "2026 Ed Brindley"
- board text added: "RCBus parallel printer adapter"
- board text added: "Rev: ${VERSION}"
- board text removed: "04 08 10 20 40 80"
- board text removed: "2017-2026 Ed Brindley"
- board text removed: "A2 A3 A4 A5 A6 A7"
- board text removed: "Active"
- board text removed: "RC2014 IDE adapter"
- board text removed: "Rev: ${VERSION} ${GIT_HASH}"
