File: rcbus-parallel.kicad_pcb (KiCad board)
At the start: 2 copper layers, 100 x 50 mm, 17 parts, among them J1 Conn_02x06_Odd_Even, J2 Conn_02x20_Odd_Even, P1 Conn_01x39, U1 82C55A_PLCC, U2 74HCT688, U3 74HCT04

Commit message: update pcb to match schematic
Connections:
- U1 pad 11: /PC7 -> unconnected-(U1-PC7-Pad11)
- U1 pad 13: /PC6 -> unconnected-(U1-PC6-Pad13)
- U1 pad 14: /PC5 -> unconnected-(U1-PC5-Pad14)
- U1 pad 15: /PC4 -> unconnected-(U1-PC4-Pad15)
Changed lines of the file:
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@@
 			(layers "*.Cu" "*.Mask")
 			(remove_unused_layers no)
-			(net "/PC7")
+			(net "unconnected-(U1-PC7-Pad11)")
 			(pinfunction "PC7_11")
 			(pintype "bidirectional+no_connect")
@@
 			(layers "*.Cu" "*.Mask")
 			(remove_unused_layers no)
-			(net "/PC6")
+			(net "unconnected-(U1-PC6-Pad13)")
 			(pinfunction "PC6_13")
 			(pintype "bidirectional+no_connect")
@@
 			(layers "*.Cu" "*.Mask")
 			(remove_unused_layers no)
-			(net "/PC5")
+			(net "unconnected-(U1-PC5-Pad14)")
 			(pinfunction "PC5_14")
 			(pintype "bidirectional+no_connect")
@@
 			(layers "*.Cu" "*.Mask")
 			(remove_unused_layers no)
-			(net "/PC4")
+			(net "unconnected-(U1-PC4-Pad15)")
 			(pinfunction "PC4_15")
 			(pintype "bidirectional+no_connect")

Commit message: minor rework
Parts:
- moved H1 2.98 mm to (65.5, 131.5)
Routing:
- net Net-(J1-Pin_12): track 38.8 -> 32.1 mm, vias 0 -> 1
- net Net-(J1-Pin_8): track 42.6 -> 36.7 mm
- net Net-(J1-Pin_6): track 42.3 -> 37.4 mm
- net Net-(J1-Pin_10): track 40.7 -> 36.1 mm, vias 0 -> 1
- net /A1: track 51.9 -> 48.4 mm
- net /PB3: track 35.0 -> 36.8 mm
- net /A2: track 29.1 -> 30.6 mm
- net Net-(J1-Pin_4): track 45.1 -> 46.1 mm
- net /~{IORQ}: track 54.1 -> 55.0 mm
- net /PB6: track 20.3 -> 19.5 mm
- net /~{PIO_CS}: track 59.3 -> 58.5 mm
- net GND: track 98.1 -> 97.4 mm
- net VCC: track 114.2 -> 113.6 mm
