File: rcbus-parallel.kicad_pcb (KiCad board)
At the start: 2 copper layers, 100 x 50 mm, 17 parts, among them J1 Conn_02x06_Odd_Even, J2 Conn_02x20_Odd_Even, P1 Conn_01x39, U1 82C55A_PLCC, U2 74HCT688, U3 74HCT04

Commit message: add some vias
Routing:
- net GND: vias 0 -> 31
